File: Grup3_Tarda_Projecte_Netejaparabrises/Comunicacions.kicad_sch (KiCad schematic)
At the start: 3 parts, among them J1 DE9_Plug_MountingHoles, J3 PROGRAMMING CON, J6 USART CON

Commit message: canvis esquematic
Parts:
- added Rterm: 120R, symbol Device:R
- added U2: TCAN1042DRQ1, symbol TCAN1042DRQ1:TCAN1042DRQ1
Connections:
- net +VCC: now also U2.3 (VCC)
- net GND: now also J1.5, U2.2 (GND)
- net CANH: now reaches J1.2
- net CANH: now also Rterm.2, U2.7 (CANH)
- net CANL: now reaches J1.3
- net CANL: now also Rterm.1, U2.6 (CANL)
- new net CANRX: U2.4 (RXD)
- new net CANTX: U2.1 (TXD)
- no-connect marks 1 -> 10
Other:
- note added: "COMM. BUS CAN"
- note added: "COMUNICACIONS"
- note added: "CONN. PROG./DEBUG"
- note added: "CONN. USART"
- note removed: "CONN PROG./DEBUG"
- note removed: "CONN USART"
- note removed: "FALTA CAN!!"
- moved on the sheet: J1, J3, J6

Commit message: canvis esquematic
Other:
- title: Projecte Netejaparabrises - Grup 3 Tarda -> Projecte Netejaparabrises - Grup 4 Tarda
Changed lines of the file:
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@@
   (paper "A4")
   (title_block
-    (title "Projecte Netejaparabrises - Grup 3 Tarda")
+    (title "Projecte Netejaparabrises - Grup 4 Tarda")
     (date "2023-03-30")
     (rev "v1.0.30032023")
