File: Grup3_Tarda_Projecte_Netejaparabrises/Grup3_Tarda_Projecte_Netejaparabrises.kicad_sch (KiCad schematic)
At the start: 0 parts

Commit message: canvis esquematic
Other:
- title: Projecte Netejaparabrises - Grup 3 Tarda -> Projecte Netejaparabrises - Grup 4 Tarda
Changed lines of the file:
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@@
   (paper "A4")
   (title_block
-    (title "Projecte Netejaparabrises - Grup 3 Tarda")
+    (title "Projecte Netejaparabrises - Grup 4 Tarda")
     (date "2023-03-30")
     (rev "v1.0.30032023")
