File: Grup3_Tarda_Projecte_Netejaparabrises/Grup3_Tarda_Projecte_Netejaparabrises.kicad_sch (KiCad schematic)
At the start: 0 parts

Commit message: Layout 3
Other:
- note added: "DRIVERS I MOTORS"
- note removed: "POTENCIA"
Changed lines of the file:
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@@
   (title_block
     (title "Projecte Netejaparabrises - Grup 4 Tarda")
-    (date "2023-04-12")
-    (rev "v1.2.12042023")
+    (date "2023-04-05")
+    (rev "v1.1.05042023")
   )
   (polyline (pts (xy 285.75 43.18) (xy 285.75 48.26))
@@
     (effects (font (size 5 5) (thickness 1) bold) (justify left bottom))
   )
-  (text "POTENCIA" (at 199.136 52.832 0)
+  (text "DRIVERS I MOTORS" (at 199.136 52.832 0)
     (effects (font (size 5 5) (thickness 1) bold) (justify left bottom))
   )
