File: Grup3_Tarda_Projecte_Netejaparabrises/Microcontrolador.kicad_sch (KiCad schematic)
At the start: 12 parts, among them IC1 PIC18F258-I_SO, J5 JP1, SW1 SW_Push, Y1 ABLS2-16.000MHZ-D4Y-T

Commit message: canvis esquematic
Parts:
- removed D5: LED_BLUE, LED_SMD:LED_0805_2012Metric, symbol Device:LED
- removed R8: 100, Resistor_SMD:R_0805_2012Metric, symbol Device:R
- removed Y1: ABLS2-16.000MHZ-D4Y-T, Crystal:XTAL_ABLS2-16.000MHZ-D4Y-T, symbol ABLS2-16.000MHZ-D4Y-T:ABLS2-16.000MHZ-D4Y-T
- added Y1: ABLS2-8.000MHZ-D4Y-T, XTAL_ABLS2-8.000MHZ-D4Y-T, symbol ABLS2-8.000MHZ-D4Y-T:ABLS2-8.000MHZ-D4Y-T
- C1, C2: value 30p -> 22p
Connections:
- net Vdd is gone; now on net +VCC: D4.2 (A), IC1.20 (VDD)
- net +VCC: no longer R7.2
- net GND: now also R7.1
- net Vledr: now also R7.2; no longer R7.1
- net XTAL1: now also Y1.1
- net XTAL2: now also Y1.2
- net CANTX: now reaches IC1.23 (RB2/CANTX/INT2)
- net CANRX: now reaches IC1.24 (RB3/CANRX)
- net DriverM2: now reaches IC1.25 (RB4)
- net PGM renamed DriverM1
- no-connect marks 17 -> 14
Other:
- note added: "MICROCONTROLADOR"
- moved on the sheet: C1, C2, C8, D4, IC1, J5, R6, R7, SW1

Commit message: canvis esquematic
Connections:
- net GND: now also IC1.19 (VSS_2)
- no-connect marks 14 -> 13
Other:
- title: Projecte Netejaparabrises - Grup 3 Tarda -> Projecte Netejaparabrises - Grup 4 Tarda
Changed lines of the file:
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@@
   (paper "A4")
   (title_block
-    (title "Projecte Netejaparabrises - Grup 3 Tarda")
+    (title "Projecte Netejaparabrises - Grup 4 Tarda")
     (date "2023-03-30")
     (rev "v1.0.30032023")
@@
   (no_connect (at 109.728 113.284))
   (no_connect (at 109.728 90.424))
-  (no_connect (at 168.148 110.744))
   (no_connect (at 168.148 103.124))
   (no_connect (at 109.728 120.904))
@@
     (stroke (width 0) (type default))
   )
+  (wire (pts (xy 168.148 110.744) (xy 169.418 110.744))
+    (stroke (width 0) (type default))
+  )
+  (wire (pts (xy 169.418 110.744) (xy 169.418 110.236))
+    (stroke (width 0) (type default))
+  )
   (wire (pts (xy 104.648 108.204) (xy 109.728 108.204))
     (stroke (width 0) (type default))
@@
   )
   (wire (pts (xy 252.984 101.854) (xy 252.984 104.394))
+    (stroke (width 0) (type default))
+  )
+  (wire (pts (xy 169.418 110.236) (xy 170.942 110.236))
     (stroke (width 0) (type default))
   )
@@
         )
       )
+    )
+  )
+  (symbol (lib_id "power:GND") (at 170.942 110.236 0) (unit 1)
+    (in_bom yes) (on_board yes) (dnp no) (fields_autoplaced)
+    (property "Reference" "#PWR042" (at 170.942 116.586 0)
+      (effects (font (size 1.27 1.27)) hide)
+    )
+    (property "Value" "GND" (at 170.942 114.808 0)
+      (effects (font (size 1.27 1.27)))
+    )
+    (property "Footprint" "" (at 170.942 110.236 0)
+      (effects (font (size 1.27 1.27)) hide)
+    )
+    (property "Datasheet" "" (at 170.942 110.236 0)
+      (effects (font (size 1.27 1.27)) hide)
+    )
+    (pin "1")
+    (instances
+      (project "Grup3_Tarda_Projecte_Netejaparabrises"
+        (path "/7ae78f34-680b-4fd9-8391-ce3e1c73c4b5/41ec4c6b-5222-4808-bf2f-f72f20229182"
+          (reference "#PWR042") (unit 1)
+        )
+      )
