File: Grup3_Tarda_Projecte_Netejaparabrises/Microcontrolador.kicad_sch (KiCad schematic)
At the start: 20 parts, among them IC1 PIC18F258-I_SO, J2 BOTONERA, J3 PROGRAMMING CON, J5 DE9_Plug_MountingHoles, J5 JP1, J6 USART CON, SW1 SW_Push, U2 TCAN1042DRQ1, Y1 ABLS2-8.000MHZ-D4Y-T

Commit message: canvis schematic 05-04-23
Parts:
- removed C8: 100n, Capacitor_SMD:C_0805_2012Metric, symbol Device:C
- removed D4: LED_RED, LED_SMD:LED_0805_2012Metric, symbol Device:LED
- removed J6: USART CON, Connector_PinSocket_2.54mm:PinSocket_1x05_P2.54mm_Vertical, symbol Connector:Conn_01x05_Pin
- removed R7: 220, Resistor_SMD:R_0805_2012Metric, symbol Device:R
- added J7: DE9_Plug_MountingHoles, symbol Connector:DE9_Plug_MountingHoles
- R1, R3, R4, R5: value R -> 22k
Connections:
- net CANH: now also J5.7; no longer J5.2
- net CANL: now also J5.2; no longer J5.3
- net GND: now also J5.6, J7.5; no longer J5.5
- net XTAL1: now also IC1.9 (OSC1/CLKI)
- net DriverLuneta: now reaches IC1.11 (RC0/T1OSO/T1CKI)
- net DriverB1: now reaches IC1.21 (RB0/INT0)
- net DriverB2: now reaches IC1.22 (RB1/INT1)
- net PWM: no longer names the net of IC1.13 (RC2/CCP1)
- net RX renamed Rx
- net Rx: now also J7.2
- net TX renamed Tx
- net Tx: now also J7.3
- no-connect marks 18 -> 22
Other:
- note removed: "BOTO 1"
- note removed: "BOTO 2"
- note removed: "BOTO 3"
- note removed: "BOTO 4"
- moved on the sheet: C1, C2, IC1, J2, J3, J5, R1, R3, R4, R5, R6, Rterm1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

Commit message: canvis schematic i README 07-04-2023
Parts:
- removed U2: TCAN1042DRQ1, symbol TCAN1042DRQ1:TCAN1042DRQ1
- added U1: TCAN1042DRQ1, Package_SO:SOIC-8_3.9x4.9mm_P1.27mm, symbol TCAN1042DRQ1:TCAN1042DRQ1
- J5, J7: footprint (none) -> Connector_Dsub:DSUB-9_Female_Horizontal_P2.77x2.84mm_EdgePinOffset4.94mm_Housed_MountingHolesOffset7.48mm
Connections:
- net +VCC: now also U1.3 (VCC)
- net CANH: now also U1.7 (CANH)
- net CANL: now also U1.6 (CANL)
- net CANRX: now also U1.4 (RXD)
- net CANTX: now also U1.1 (TXD)
- net GND: now also U1.2 (GND)
Changed lines of the file:
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@@
-    )
-  )
-  (symbol (lib_id "Device:C") (at 106.172 132.842 0) (unit 1)
-    (in_bom yes) (on_board yes) (dnp no) (fields_autoplaced)
-    (property "Reference" "C2" (at 109.982 132.207 0)
-      (effects (font (size 1.27 1.27)) (justify left))
-    )
-    (property "Value" "22p" (at 109.982 134.747 0)
-      (effects (font (size 1.27 1.27)) (justify left))
-    )
-    (property "Footprint" "Capacitor_SMD:C_0805_2012Metric" (at 107.1372 136.652 0)
-      (effects (font (size 1.27 1.27)) hide)
-    )
-    (property "Datasheet" "~" (at 106.172 132.842 0)
-      (effects (font (size 1.27 1.27)) hide)
-    )
-    (pin "1")
-    (pin "2")
-    (instances
-      (project "Grup3_Tarda_Projecte_Netejaparabrises"
-        (path "/7ae78f34-680b-4fd9-8391-ce3e1c73c4b5"
-          (reference "C2") (unit 1)
-        )
-        (path "/7ae78f34-680b-4fd9-8391-ce3e1c73c4b5/41ec4c6b-5222-4808-bf2f-f72f20229182"
-          (reference "C?") (unit 1)
-        )
-      )
-      (project "AidarIglesias_DavidMiravent_P3"
-        (path "/f9f603a9-b774-48a7-94d1-4c8d3d65a3f8"
-          (reference "C2") (unit 1)
-        )
-      )
-    )
-  )
-  (symbol (lib_id "Device:R") (at 44.704 119.634 0) (unit 1)
-    (in_bom yes) (on_board yes) (dnp no)
-    (property "Reference" "R3" (at 39.624 118.364 0)
-      (effects (font (size 1.27 1.27)) (justify left))
-    )
-    (property "Value" "22k" (at 39.624 120.904 0)
-      (effects (font (size 1.27 1.27)) (justify left))
-    )
-    (property "Footprint" "" (at 42.926 119.634 90)
-      (effects (font (size 1.27 1.27)) hide)
-    )
-    (property "Datasheet" "~" (at 44.704 119.634 0)
-      (effects (font (size 1.27 1.27)) hide)
-    )
-    (pin "1")
-    (pin "2")
-    (instances
-      (project "Grup3_Tarda_Projecte_Netejaparabrises"
-        (path "/7ae78f34-680b-4fd9-8391-ce3e1c73c4b5/41ec4c6b-5222-4808-bf2f-f72f20229182"
-          (reference "R3") (unit 1)
-        )
-      )
-    )
-  )
-  (symbol (lib_id "Device:C") (at 88.646 132.842 0) (unit 1)
-    (in_bom yes) (on_board yes) (dnp no) (fields_autoplaced)
-    (property "Reference" "C1" (at 92.456 132.207 0)
-      (effects (font (size 1.27 1.27)) (justify left))
-    )
-    (property "Value" "22p" (at 92.456 134.747 0)
-      (effects (font (size 1.27 1.27)) (justify left))
-    )
-    (property "Footprint" "Capacitor_SMD:C_0805_2012Metric" (at 89.6112 136.652 0)
-      (effects (font (size 1.27 1.27)) hide)
-    )
-    (property "Datasheet" "~" (at 88.646 132.842 0)
-      (effects (font (size 1.27 1.27)) hide)
-    )
-    (pin "1")
-    (pin "2")
-    (instances
-      (project "Grup3_Tarda_Projecte_Netejaparabrises"
-        (path "/7ae78f34-680b-4fd9-8391-ce3e1c73c4b5"
-          (reference "C1") (unit 1)
-        )
-        (path "/7ae78f34-680b-4fd9-8391-ce3e1c73c4b5/41ec4c6b-5222-4808-bf2f-f72f20229182"
-          (reference "C?") (unit 1)
-        )
-      )
-      (project "AidarIglesias_DavidMiravent_P3"
-        (path "/f9f603a9-b774-48a7-94d1-4c8d3d65a3f8"
-          (reference "C1") (unit 1)
-        )
-      )
     )
   )
   (symbol (lib_id "TCAN1042DRQ1:TCAN1042DRQ1") (at 216.408 97.79 0) (unit 1)
     (in_bom yes) (on_board yes) (dnp no) (fields_autoplaced)
-    (property "Reference" "U2" (at 216.408 86.106 0)
-      (effects (font (size 1.27 1.27)))
-    )
-    (property "Value" "TCAN1042DRQ1" (at 216.408 88.646 0)
-      (effects (font (size 1.27 1.27)))
-    )
-    (property "Footprint" "" (at 216.408 97.79 0)
+    (property "Reference" "U1" (at 216.408 86.36 0)
+      (effects (font (size 1.27 1.27)))
+    )
+    (property "Value" "TCAN1042DRQ1" (at 216.408 88.9 0)
+      (effects (font (size 1.27 1.27)))
+    )
+    (property "Footprint" "Package_SO:SOIC-8_3.9x4.9mm_P1.27mm" (at 216.408 97.79 0)
       (effects (font (size 1.27 1.27)) hide)
     )
@@
       (project "Grup3_Tarda_Projecte_Netejaparabrises"
         (path "/7ae78f34-680b-4fd9-8391-ce3e1c73c4b5/41ec4c6b-5222-4808-bf2f-f72f20229182"
-          (reference "U2") (unit 1)
+          (reference "U1") (unit 1)
+        )
+      )
+    )
+  )
+  (symbol (lib_id "Device:C") (at 106.172 132.842 0) (unit 1)
+    (in_bom yes) (on_board yes) (dnp no) (fields_autoplaced)
+    (property "Reference" "C2" (at 109.982 132.207 0)
+      (effects (font (size 1.27 1.27)) (justify left))
+    )
+    (property "Value" "22p" (at 109.982 134.747 0)
+      (effects (font (size 1.27 1.27)) (justify left))
+    )
+    (property "Footprint" "Capacitor_SMD:C_0805_2012Metric" (at 107.1372 136.652 0)
+      (effects (font (size 1.27 1.27)) hide)
+    )
+    (property "Datasheet" "~" (at 106.172 132.842 0)
+      (effects (font (size 1.27 1.27)) hide)
+    )
+    (pin "1")
+    (pin "2")
+    (instances
+      (project "Grup3_Tarda_Projecte_Netejaparabrises"
+        (path "/7ae78f34-680b-4fd9-8391-ce3e1c73c4b5"
+          (reference "C2") (unit 1)
+        )
+        (path "/7ae78f34-680b-4fd9-8391-ce3e1c73c4b5/41ec4c6b-5222-4808-bf2f-f72f20229182"
+          (reference "C?") (unit 1)
+        )
+      )
+      (project "AidarIglesias_DavidMiravent_P3"
+        (path "/f9f603a9-b774-48a7-94d1-4c8d3d65a3f8"
+          (reference "C2") (unit 1)
+        )
+      )
+    )
+  )
+  (symbol (lib_id "Device:R") (at 44.704 119.634 0) (unit 1)
+    (in_bom yes) (on_board yes) (dnp no)
+    (property "Reference" "R3" (at 39.624 118.364 0)
+      (effects (font (size 1.27 1.27)) (justify left))
+    )
+    (property "Value" "22k" (at 39.624 120.904 0)
+      (effects (font (size 1.27 1.27)) (justify left))
+    )
+    (property "Footprint" "" (at 42.926 119.634 90)
+      (effects (font (size 1.27 1.27)) hide)
+    )
+    (property "Datasheet" "~" (at 44.704 119.634 0)
+      (effects (font (size 1.27 1.27)) hide)
+    )
+    (pin "1")
+    (pin "2")
+    (instances
+      (project "Grup3_Tarda_Projecte_Netejaparabrises"
+        (path "/7ae78f34-680b-4fd9-8391-ce3e1c73c4b5/41ec4c6b-5222-4808-bf2f-f72f20229182"
+          (reference "R3") (unit 1)
+        )
+      )
+    )
+  )
+  (symbol (lib_id "Device:C") (at 88.646 132.842 0) (unit 1)
+    (in_bom yes) (on_board yes) (dnp no) (fields_autoplaced)
+    (property "Reference" "C1" (at 92.456 132.207 0)
+      (effects (font (size 1.27 1.27)) (justify left))
+    )
+    (property "Value" "22p" (at 92.456 134.747 0)
+      (effects (font (size 1.27 1.27)) (justify left))
+    )
+    (property "Footprint" "Capacitor_SMD:C_0805_2012Metric" (at 89.6112 136.652 0)
+      (effects (font (size 1.27 1.27)) hide)
+    )
+    (property "Datasheet" "~" (at 88.646 132.842 0)
+      (effects (font (size 1.27 1.27)) hide)
+    )
+    (pin "1")
+    (pin "2")
+    (instances
+      (project "Grup3_Tarda_Projecte_Netejaparabrises"
+        (path "/7ae78f34-680b-4fd9-8391-ce3e1c73c4b5"
+          (reference "C1") (unit 1)
+        )
+        (path "/7ae78f34-680b-4fd9-8391-ce3e1c73c4b5/41ec4c6b-5222-4808-bf2f-f72f20229182"
+          (reference "C?") (unit 1)
+        )
+      )
+      (project "AidarIglesias_DavidMiravent_P3"
+        (path "/f9f603a9-b774-48a7-94d1-4c8d3d65a3f8"
+          (reference "C1") (unit 1)
         )
       )
@@
       (effects (font (size 1.27 1.27)) (justify left))
     )
-    (property "Footprint" "" (at 211.074 122.682 0)
+    (property "Footprint" "Connector_Dsub:DSUB-9_Female_Horizontal_P2.77x2.84mm_EdgePinOffset4.94mm_Housed_MountingHolesOffset7.48mm" (at 211.074 122.682 0)
       (effects (font (size 1.27 1.27)) hide)
     )
@@
       (effects (font (size 1.27 1.27)) (justify left))
     )
-    (property "Footprint" "" (at 252.476 97.79 0)
-      (effects (font (size 1.27 1.27)) hide)
-    )
+    (property "Footprint" "Connector_Dsub:DSUB-9_Female_Horizontal_P2.77x2.84mm_EdgePinOffset4.94mm_Housed_MountingHolesOffset7.48mm" (at 252.476 97.79 0)
+      (effects (font (size 1.27 1.27)) hide)
+    )

Commit message: canvis reles 07-04-2023
Connections:
- net EnableM1: now reaches IC1.12 (RC1/T1OSI)
- net EnableM2: now reaches IC1.13 (RC2/CCP1)
- no-connect marks 22 -> 20
Other:
- note added: "DIGITAL"
- note removed: "MICROCONTROLADOR"
- moved on the sheet: C1, C2, Y1

Commit message: GNDS 08042023
Changed lines of the file:
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@@
       (effects (font (size 1.27 1.27)) hide)
     )
-    (property "Value" "GND" (at 91.44 143.764 0)
-      (effects (font (size 1.27 1.27)))
+    (property "Value" "GND3" (at 93.98 140.589 0)
+      (effects (font (size 1.27 1.27)) (justify left))
     )
     (property "Footprint" "" (at 91.44 138.684 0)
@@
       (effects (font (size 1.27 1.27)) hide)
     )
-    (property "Value" "GND" (at 37.338 70.231 0)
+    (property "Value" "GND2" (at 36.83 70.231 0)
       (effects (font (size 1.27 1.27)) (justify left))
     )
@@
       (effects (font (size 1.27 1.27)) hide)
     )
-    (property "Value" "GND" (at 29.718 146.812 0)
-      (effects (font (size 1.27 1.27)))
+    (property "Value" "GND2" (at 31.75 143.637 0)
+      (effects (font (size 1.27 1.27)) (justify left))
     )
     (property "Footprint" "" (at 29.718 141.732 0)
@@
       (effects (font (size 1.27 1.27)) hide)
     )
-    (property "Value" "GND" (at 35.814 138.684 0)
-      (effects (font (size 1.27 1.27)))
+    (property "Value" "GND2" (at 38.1 135.509 0)
+      (effects (font (size 1.27 1.27)) (justify left))
     )
     (property "Footprint" "" (at 35.814 133.604 0)
@@
       (effects (font (size 1.27 1.27)) hide)
     )
-    (property "Value" "GND" (at 101.854 77.47 0)
-      (effects (font (size 1.27 1.27)))
+    (property "Value" "GND2" (at 104.14 74.295 0)
+      (effects (font (size 1.27 1.27)) (justify left))
     )
     (property "Footprint" "" (at 101.854 72.39 0)
@@
       (effects (font (size 1.27 1.27)) hide)
     )
-    (property "Value" "GND" (at 200.152 118.364 0)
-      (effects (font (size 1.27 1.27)))
+    (property "Value" "GND2" (at 203.2 115.697 0)
+      (effects (font (size 1.27 1.27)) (justify left))
     )
     (property "Footprint" "" (at 200.152 113.792 0)
@@
       (effects (font (size 1.27 1.27)) hide)
     )
-    (property "Value" "GND" (at 231.648 90.424 0)
-      (effects (font (size 1.27 1.27)))
+    (property "Value" "GND2" (at 233.68 87.757 0)
+      (effects (font (size 1.27 1.27)) (justify left))
     )
     (property "Footprint" "" (at 231.648 85.852 0)
@@
       (effects (font (size 1.27 1.27)) hide)
     )
-    (property "Value" "GND" (at 107.442 112.014 0)
-      (effects (font (size 1.27 1.27)))
+    (property "Value" "GND2" (at 110.49 108.839 0)
+      (effects (font (size 1.27 1.27)) (justify left))
     )
     (property "Footprint" "" (at 107.442 106.934 0)
@@
       (effects (font (size 1.27 1.27)) hide)
     )
-    (property "Value" "GND" (at 176.276 108.458 0)
-      (effects (font (size 1.27 1.27)))
+    (property "Value" "GND2" (at 179.07 105.791 0)
+      (effects (font (size 1.27 1.27)) (justify left))
     )
     (property "Footprint" "" (at 176.276 103.886 0)

Commit message: definitiuEsquematicsenseFootprints
Parts:
- added C2 (x2): 100n, Capacitor_SMD:C_0805_2012Metric, symbol Device:C
- renumbered R1 to RBot1, R3 to RBot2, R4 to RBot3, R5 to RBot4
Connections:
- net +VCC: now also C2.1, C2.1
- net GND: now also C2.2, C2.2
Other:
- moved on the sheet: J7

Commit message: Layout Esquema
Parts:
- renumbered J7 to J5, J5 to J6
Changed lines of the file:
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@@
   (symbol (lib_id "power:GND") (at 91.44 138.684 0) (unit 1)
     (in_bom yes) (on_board yes) (dnp no) (fields_autoplaced)
-    (property "Reference" "#PWR05" (at 91.44 145.034 0)
+    (property "Reference" "#PWR09" (at 91.44 145.034 0)
       (effects (font (size 1.27 1.27)) hide)
     )
@@
       (project "Grup3_Tarda_Projecte_Netejaparabrises"
         (path "/7ae78f34-680b-4fd9-8391-ce3e1c73c4b5/41ec4c6b-5222-4808-bf2f-f72f20229182"
-          (reference "#PWR05") (unit 1)
+          (reference "#PWR09") (unit 1)
         )
       )
@@
         )
         (path "/7ae78f34-680b-4fd9-8391-ce3e1c73c4b5/41ec4c6b-5222-4808-bf2f-f72f20229182"
-          (reference "#PWR08") (unit 1)
+          (reference "#PWR07") (unit 1)
         )
       )
@@
   (symbol (lib_id "power:GND") (at 29.718 141.732 0) (unit 1)
     (in_bom yes) (on_board yes) (dnp no) (fields_autoplaced)
-    (property "Reference" "#PWR013" (at 29.718 148.082 0)
+    (property "Reference" "#PWR06" (at 29.718 148.082 0)
       (effects (font (size 1.27 1.27)) hide)
     )
@@
       (project "Grup3_Tarda_Projecte_Netejaparabrises"
         (path "/7ae78f34-680b-4fd9-8391-ce3e1c73c4b5/41ec4c6b-5222-4808-bf2f-f72f20229182"
-          (reference "#PWR013") (unit 1)
+          (reference "#PWR06") (unit 1)
         )
       )
@@
         )
         (path "/7ae78f34-680b-4fd9-8391-ce3e1c73c4b5/41ec4c6b-5222-4808-bf2f-f72f20229182"
-          (reference "CDesacobCan") (unit 1)
+          (reference "CDesacobCan1") (unit 1)
         )
       )
@@
         )
         (path "/7ae78f34-680b-4fd9-8391-ce3e1c73c4b5/41ec4c6b-5222-4808-bf2f-f72f20229182"
-          (reference "J1") (unit 1)
-        )
-      )
-      (project "AidarIglesias_DavidMiravent_P3"
-        (path "/f9f603a9-b774-48a7-94d1-4c8d3d65a3f8"
           (reference "J3") (unit 1)
         )
       )
+      (project "AidarIglesias_DavidMiravent_P3"
+        (path "/f9f603a9-b774-48a7-94d1-4c8d3d65a3f8"
+          (reference "J3") (unit 1)
+        )
+      )
     )
   )
   (symbol (lib_id "power:GND") (at 35.814 133.604 0) (unit 1)
     (in_bom yes) (on_board yes) (dnp no) (fields_autoplaced)
-    (property "Reference" "#PWR024" (at 35.814 139.954 0)
+    (property "Reference" "#PWR08" (at 35.814 139.954 0)
       (effects (font (size 1.27 1.27)) hide)
     )
@@
       (project "Grup3_Tarda_Projecte_Netejaparabrises"
         (path "/7ae78f34-680b-4fd9-8391-ce3e1c73c4b5/41ec4c6b-5222-4808-bf2f-f72f20229182"
-          (reference "#PWR024") (unit 1)
+          (reference "#PWR08") (unit 1)
         )
       )
@@
         )
         (path "/7ae78f34-680b-4fd9-8391-ce3e1c73c4b5/41ec4c6b-5222-4808-bf2f-f72f20229182"
-          (reference "SWReset") (unit 1)
+          (reference "SWReset1") (unit 1)
         )
       )
@@
         )
         (path "/7ae78f34-680b-4fd9-8391-ce3e1c73c4b5/41ec4c6b-5222-4808-bf2f-f72f20229182"
-          (reference "#PWR022") (unit 1)
+          (reference "#PWR010") (unit 1)
         )
       )
@@
         )
         (path "/7ae78f34-680b-4fd9-8391-ce3e1c73c4b5/41ec4c6b-5222-4808-bf2f-f72f20229182"
-          (reference "CDesacobMicro") (unit 1)
+          (reference "CDesacobMicro1") (unit 1)
         )
       )
@@
         )
         (path "/7ae78f34-680b-4fd9-8391-ce3e1c73c4b5/41ec4c6b-5222-4808-bf2f-f72f20229182"
-          (reference "RReset") (unit 1)
+          (reference "RReset1") (unit 1)
         )
       )
@@
         )
         (path "/7ae78f34-680b-4fd9-8391-ce3e1c73c4b5/41ec4c6b-5222-4808-bf2f-f72f20229182"
-          (reference "#PWR02") (unit 1)
+          (reference "#PWR015") (unit 1)
         )
       )
@@
   (symbol (lib_id "power:GND") (at 192.532 116.967 0) (unit 1)
     (in_bom yes) (on_board yes) (dnp no)
-    (property "Reference" "#PWR043" (at 192.532 123.317 0)
+    (property "Reference" "#PWR013" (at 192.532 123.317 0)
       (effects (font (size 1.27 1.27)) hide)
     )
@@
       (project "Grup3_Tarda_Projecte_Netejaparabrises"
         (path "/7ae78f34-680b-4fd9-8391-ce3e1c73c4b5/41ec4c6b-5222-4808-bf2f-f72f20229182"
-          (reference "#PWR043") (unit 1)
+          (reference "#PWR013") (unit 1)
         )
       )
@@
   (symbol (lib_id "power:GND") (at 231.648 85.852 0) (unit 1)
     (in_bom yes) (on_board yes) (dnp no) (fields_autoplaced)
-    (property "Reference" "#PWR04" (at 231.648 92.202 0)
+    (property "Reference" "#PWR016" (at 231.648 92.202 0)
       (effects (font (size 1.27 1.27)) hide)
     )
@@
       (project "Grup3_Tarda_Projecte_Netejaparabrises"
         (path "/7ae78f34-680b-4fd9-8391-ce3e1c73c4b5/41ec4c6b-5222-4808-bf2f-f72f20229182"
-          (reference "#PWR04") (unit 1)
+          (reference "#PWR016") (unit 1)
         )
       )
@@
   (symbol (lib_id "power:GND") (at 201.676 117.729 0) (unit 1)
     (in_bom yes) (on_board yes) (dnp no)
-    (property "Reference" "#PWR044" (at 201.676 124.079 0)
+    (property "Reference" "#PWR014" (at 201.676 124.079 0)
       (effects (font (size 1.27 1.27)) hide)
     )
@@
       (project "Grup3_Tarda_Projecte_Netejaparabrises"
         (path "/7ae78f34-680b-4fd9-8391-ce3e1c73c4b5/41ec4c6b-5222-4808-bf2f-f72f20229182"
-          (reference "#PWR044") (unit 1)
+          (reference "#PWR014") (unit 1)
         )
       )
@@
         )
         (path "/7ae78f34-680b-4fd9-8391-ce3e1c73c4b5/41ec4c6b-5222-4808-bf2f-f72f20229182"
-          (reference "IC?") (unit 1)
+          (reference "IC2") (unit 1)
         )
       )
@@
   (symbol (lib_id "Connector:DE9_Plug_MountingHoles") (at 229.616 138.938 0) (unit 1)
     (in_bom yes) (on_board yes) (dnp no) (fields_autoplaced)
-    (property "Reference" "J7" (at 234.188 138.303 0)
+    (property "Reference" "J5" (at 234.188 138.303 0)
       (effects (font (size 1.27 1.27)) (justify left))
     )
@@
       (project "Grup3_Tarda_Projecte_Netejaparabrises"
         (path "/7ae78f34-680b-4fd9-8391-ce3e1c73c4b5/41ec4c6b-5222-4808-bf2f-f72f20229182"
-          (reference "J7") (unit 1)
+          (reference "J5") (unit 1)
         )
       )
@@
         )
         (path "/7ae78f34-680b-4fd9-8391-ce3e1c73c4b5/41ec4c6b-5222-4808-bf2f-f72f20229182"
-          (reference "J?") (unit 1)
+          (reference "J4") (unit 1)
         )
       )
@@
   (symbol (lib_id "Connector:DE9_Plug_MountingHoles") (at 252.476 97.79 0) (mirror x) (unit 1)
     (in_bom yes) (on_board yes) (dnp no)
-    (property "Reference" "J5" (at 257.048 98.425 0)
+    (property "Reference" "J6" (at 257.048 98.425 0)
       (effects (font (size 1.27 1.27)) (justify left))
     )
@@
       (project "Grup3_Tarda_Projecte_Netejaparabrises"
         (path "/7ae78f34-680b-4fd9-8391-ce3e1c73c4b5/41ec4c6b-5222-4808-bf2f-f72f20229182"
-          (reference "J5") (unit 1)
+          (reference "J6") (unit 1)
         )
       )
@@
   (symbol (lib_id "power:GND") (at 186.436 113.792 0) (unit 1)
     (in_bom yes) (on_board yes) (dnp no)
-    (property "Reference" "#PWR042" (at 186.436 120.142 0)
+    (property "Reference" "#PWR012" (at 186.436 120.142 0)
       (effects (font (size 1.27 1.27)) hide)
     )
@@
       (project "Grup3_Tarda_Projecte_Netejaparabrises"
         (path "/7ae78f34-680b-4fd9-8391-ce3e1c73c4b5/41ec4c6b-5222-4808-bf2f-f72f20229182"
-          (reference "#PWR042") (unit 1)
-        )
-      )
+          (reference "#PWR012") (unit 1)
+        )
+      )
