File: Grup3_Tarda_Projecte_Netejaparabrises/Potencia.kicad_sch (KiCad schematic)
At the start: 43 parts, among them J6 CONNECTOR ALIMENTACIO, K1 1393280-6, K2 1393280-6, K3 1393280-6, K4 1393280-6, K5 1393280-6, K6 1393280-6, K8 1393280-6, Q1 BC817-25_RF, Q2 BC817-25_RF, Q3 BC817-25_RF, Q4 BC817-25_RF, Q5 BC817-25_RF, Q6 BC817-25_RF, Q7 BC817-25_RF

Commit message: canvis schematic 05-04-23
Connections:
- net VMOT2+: no longer J6.4 (Pin_4), K3.5
- new net VMOT2-: J6.4 (Pin_4), K3.5
Other:
- note added: "DRIVER BOMBES"
- note added: "DRIVER MOTOR DARRERE"
- note added: "DRIVER MOTOR DAVANT"
- note removed: "DRIVER BOMBAS"
- note removed: "DRIVER MOTOR 1"
- note removed: "DRIVER MOTOR 2"

Commit message: canvis schematic i README 07-04-2023
Connections:
- net VBAT: now also K1.5, K2.5, K3.5, K4.5, K5.5, K6.5, K8.5; no longer K1.4, K2.4, K3.4, K4.4, K5.4, K6.4, K8.4
- net VBOMBA1: now also K4.4; no longer K4.5
- net VBOMBA2: now also K5.4; no longer K5.5
- net VLUNETA: now also K6.4; no longer K6.5
- net VMOT1+: now also K1.4; no longer K1.5
- net VMOT1-: now also K8.4; no longer K8.5
- net VMOT2+: now also K2.4; no longer K2.5
- net VMOT2-: now also K3.4; no longer K3.5
Changed lines of the file:
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@@
     )
   )
-  (global_label "VMOT2+" (shape output) (at 210.312 33.528 0) (fields_autoplaced)
+  (global_label "VMOT2+" (shape output) (at 211.328 38.608 0) (fields_autoplaced)
     (effects (font (size 1.27 1.27)) (justify left))
-    (property "Intersheetrefs" "${INTERSHEET_REFS}" (at 220.8378 33.528 0)
+    (property "Intersheetrefs" "${INTERSHEET_REFS}" (at 221.8538 38.608 0)
       (effects (font (size 1.27 1.27)) (justify left) hide)
     )
   )
-  (global_label "VBAT" (shape input) (at 118.872 75.184 0) (fields_autoplaced)
+  (global_label "VBAT" (shape input) (at 118.618 70.104 0) (fields_autoplaced)
     (effects (font (size 1.27 1.27)) (justify left))
-    (property "Intersheetrefs" "${INTERSHEET_REFS}" (at 126.1926 75.184 0)
+    (property "Intersheetrefs" "${INTERSHEET_REFS}" (at 125.9386 70.104 0)
       (effects (font (size 1.27 1.27)) (justify left) hide)
     )
   )
-  (global_label "VBAT" (shape input) (at 256.794 72.39 0) (fields_autoplaced)
+  (global_label "VBAT" (shape input) (at 260.096 67.31 0) (fields_autoplaced)
     (effects (font (size 1.27 1.27)) (justify left))
-    (property "Intersheetrefs" "${INTERSHEET_REFS}" (at 264.1146 72.39 0)
+    (property "Intersheetrefs" "${INTERSHEET_REFS}" (at 267.4166 67.31 0)
       (effects (font (size 1.27 1.27)) (justify left) hide)
     )
@@
     )
   )
-  (global_label "VBAT" (shape input) (at 257.302 135.382 0) (fields_autoplaced)
+  (global_label "VBAT" (shape input) (at 256.794 130.302 0) (fields_autoplaced)
     (effects (font (size 1.27 1.27)) (justify left))
-    (property "Intersheetrefs" "${INTERSHEET_REFS}" (at 264.6226 135.382 0)
+    (property "Intersheetrefs" "${INTERSHEET_REFS}" (at 264.1146 130.302 0)
       (effects (font (size 1.27 1.27)) (justify left) hide)
     )
@@
     )
   )
-  (global_label "VMOT1+" (shape output) (at 81.788 34.544 0) (fields_autoplaced)
+  (global_label "VMOT1+" (shape output) (at 82.296 39.624 0) (fields_autoplaced)
     (effects (font (size 1.27 1.27)) (justify left))
-    (property "Intersheetrefs" "${INTERSHEET_REFS}" (at 92.3138 34.544 0)
+    (property "Intersheetrefs" "${INTERSHEET_REFS}" (at 92.8218 39.624 0)
       (effects (font (size 1.27 1.27)) (justify left) hide)
     )
   )
-  (global_label "VBOMBA1" (shape output) (at 83.312 137.414 0) (fields_autoplaced)
+  (global_label "VBOMBA1" (shape output) (at 83.82 142.494 0) (fields_autoplaced)
     (effects (font (size 1.27 1.27)) (justify left))
-    (property "Intersheetrefs" "${INTERSHEET_REFS}" (at 94.9264 137.414 0)
+    (property "Intersheetrefs" "${INTERSHEET_REFS}" (at 95.4344 142.494 0)
       (effects (font (size 1.27 1.27)) (justify left) hide)
     )
   )
-  (global_label "VBAT" (shape input) (at 83.82 142.494 0) (fields_autoplaced)
+  (global_label "VBAT" (shape input) (at 83.312 137.414 0) (fields_autoplaced)
     (effects (font (size 1.27 1.27)) (justify left))
-    (property "Intersheetrefs" "${INTERSHEET_REFS}" (at 91.1406 142.494 0)
+    (property "Intersheetrefs" "${INTERSHEET_REFS}" (at 90.6326 137.414 0)
       (effects (font (size 1.27 1.27)) (justify left) hide)
     )
   )
-  (global_label "VBAT" (shape input) (at 211.328 38.608 0) (fields_autoplaced)
+  (global_label "VBAT" (shape input) (at 210.312 33.528 0) (fields_autoplaced)
     (effects (font (size 1.27 1.27)) (justify left))
-    (property "Intersheetrefs" "${INTERSHEET_REFS}" (at 218.6486 38.608 0)
+    (property "Intersheetrefs" "${INTERSHEET_REFS}" (at 217.6326 33.528 0)
       (effects (font (size 1.27 1.27)) (justify left) hide)
     )
@@
     )
   )
-  (global_label "VBAT" (shape input) (at 154.686 141.986 0) (fields_autoplaced)
+  (global_label "VBAT" (shape input) (at 154.178 136.906 0) (fields_autoplaced)
     (effects (font (size 1.27 1.27)) (justify left))
-    (property "Intersheetrefs" "${INTERSHEET_REFS}" (at 162.0066 141.986 0)
+    (property "Intersheetrefs" "${INTERSHEET_REFS}" (at 161.4986 136.906 0)
       (effects (font (size 1.27 1.27)) (justify left) hide)
     )
@@
     )
   )
-  (global_label "VMOT1-" (shape output) (at 118.618 70.104 0) (fields_autoplaced)
+  (global_label "VMOT1-" (shape output) (at 118.872 75.184 0) (fields_autoplaced)
     (effects (font (size 1.27 1.27)) (justify left))
-    (property "Intersheetrefs" "${INTERSHEET_REFS}" (at 129.1438 70.104 0)
+    (property "Intersheetrefs" "${INTERSHEET_REFS}" (at 129.3978 75.184 0)
       (effects (font (size 1.27 1.27)) (justify left) hide)
     )
   )
-  (global_label "VBOMBA2" (shape output) (at 154.178 136.906 0) (fields_autoplaced)
+  (global_label "VBOMBA2" (shape output) (at 154.686 141.986 0) (fields_autoplaced)
     (effects (font (size 1.27 1.27)) (justify left))
-    (property "Intersheetrefs" "${INTERSHEET_REFS}" (at 165.7924 136.906 0)
+    (property "Intersheetrefs" "${INTERSHEET_REFS}" (at 166.3004 141.986 0)
       (effects (font (size 1.27 1.27)) (justify left) hide)
     )
@@
     )
   )
-  (global_label "VMOT2-" (shape output) (at 260.096 67.31 0) (fields_autoplaced)
+  (global_label "VMOT2-" (shape output) (at 256.794 72.39 0) (fields_autoplaced)
     (effects (font (size 1.27 1.27)) (justify left))
-    (property "Intersheetrefs" "${INTERSHEET_REFS}" (at 270.6218 67.31 0)
+    (property "Intersheetrefs" "${INTERSHEET_REFS}" (at 267.3198 72.39 0)
       (effects (font (size 1.27 1.27)) (justify left) hide)
     )
@@
     )
   )
-  (global_label "VBAT" (shape input) (at 82.296 39.624 0) (fields_autoplaced)
+  (global_label "VBAT" (shape input) (at 81.788 34.544 0) (fields_autoplaced)
     (effects (font (size 1.27 1.27)) (justify left))
-    (property "Intersheetrefs" "${INTERSHEET_REFS}" (at 89.6166 39.624 0)
+    (property "Intersheetrefs" "${INTERSHEET_REFS}" (at 89.1086 34.544 0)
       (effects (font (size 1.27 1.27)) (justify left) hide)
     )
   )
-  (global_label "VLUNETA" (shape output) (at 256.794 130.302 0) (fields_autoplaced)
+  (global_label "VLUNETA" (shape output) (at 257.302 135.382 0) (fields_autoplaced)
     (effects (font (size 1.27 1.27)) (justify left))
-    (property "Intersheetrefs" "${INTERSHEET_REFS}" (at 267.6827 130.302 0)
+    (property "Intersheetrefs" "${INTERSHEET_REFS}" (at 268.1907 135.382 0)
       (effects (font (size 1.27 1.27)) (justify left) hide)
     )

Commit message: canvis reles 07-04-2023
Parts:
- removed J6: CONNECTOR ALIMENTACIO, symbol Connector:Conn_01x07_Pin
- added D10, D9: 1N5400, Diode_THT:D_DO-201AD_P15.24mm_Horizontal, symbol Diode:1N5400
- added J4: CONNECTOR ALIMENTACIO, symbol Connector:Conn_01x10_Pin
- added K7, K9: 1393280-6, RELAY_1393280-6, symbol 1393280-6:1393280-6
Connections:
- net DriverM1: no longer R10.1
- net DriverM2: no longer R16.1
- net GND: now also K8.5, J4.10 (Pin_10), J4.6 (Pin_6), J4.8 (Pin_8), K7.3, K9.3; no longer K8.3
- net VBAT: now also D10.1 (K), D9.1 (K), K7.1, K7.5, K9.1, K9.5; no longer K1.5, K2.5, K3.5, K8.5
- net VBOMBA1: now also J4.5 (Pin_5)
- net VBOMBA2: now also J4.7 (Pin_7)
- net VLUNETA: now also J4.9 (Pin_9)
- net VMOT1+: now also J4.1 (Pin_1)
- net VMOT1-: now also J4.2 (Pin_2)
- net VMOT2+: now also J4.3 (Pin_3)
- net VMOT2-: now also J4.4 (Pin_4)
- net Vb_m1+ renamed Vb_m1
- net Vb_m1- renamed Vb_EN1
- net Vb_m2+ renamed Vb_m2
- net Vb_m2- renamed Vb_EN2
- net Vc_m1+ renamed Vc_m1
- net Vc_m1: now also D2.2 (A), K8.2
- removed net Vc_m1-: D2.2 (A), K8.2, Q2.3
- net Vc_m2+ renamed Vc_m2
- net Vc_m2: now also D4.2 (A), K3.2
- removed net Vc_m2-: D4.2 (A), K3.2, Q4.3
- net Ve_m1+ renamed Ve_m1
- net Ve_m1- renamed Ve_EN1
- net Ve_m2+ renamed Ve_m2
- net Ve_m2- renamed Ve_EN2
- new net EN1: K1.5, K7.4, K8.3
- new net EN2: K2.5, K3.5, K9.4
- new net EnableM1: R10.1
- new net EnableM2: R16.1
- new net Vc_EN1: D9.2 (A), K7.2, Q2.3
- new net Vc_EN2: D10.2 (A), K9.2, Q4.3
Other:
- moved on the sheet: D1, D2, D3, D4, D5, D6, D7, K1, K2, K3, K4, K5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

Commit message: GNDS 08042023
Connections:
- net GND renamed GNDPWR

Commit message: Layout Esquema
Parts:
- renumbered D3 to D10, D4 to D11, D7 to D12, D5 to D4, D9 to D5, D1 to D6, D2 to D7, D6 to D8, D10 to D9, J4 to J8, K4 to K1, K7 to K2, K1 to K3, K8 to K4, K9 to K6, K3 to K7, K2 to K8, K6 to K9, Q5 to Q1, Q1 to Q3, Q6 to Q4, Q4 to Q5, Q3 to Q6, R9 to R10, R22 to R11, R23 to R12, R24 to R13, R16 to R14, R13 to R15, R17 to R16, R14 to R17, R15 to R19, R19 to R2, R25 to R20, R26 to R21, R27 to R22, R10 to R3, R7 to R4, R20 to R5, R11 to R6, R8 to R7, R21 to R8, R12 to R9
