File: Grup3_Tarda_Projecte_Netejaparabrises/Sensor_Pluja.kicad_sch (KiCad schematic)
At the start: 5 parts, among them J3 CONEXIOSENSOR, U3 LM393

Commit message: Layout Esquema
Parts:
- CDesOpam1: renamed from CDesOpam; footprint (none) -> Capacitor_SMD:CP_Elec_4x3
- renumbered J3 to J7, RPOT to RPOT1, RSens to RSens1, U3 to U2
Changed lines of the file:
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@@
   (symbol (lib_id "Connector:Conn_01x02_Pin") (at 88.9 99.06 0) (unit 1)
     (in_bom yes) (on_board yes) (dnp no)
-    (property "Reference" "J3" (at 89.408 92.456 0)
+    (property "Reference" "J7" (at 89.408 92.456 0)
       (effects (font (size 1.27 1.27)))
     )
@@
       (project "Grup3_Tarda_Projecte_Netejaparabrises"
         (path "/7ae78f34-680b-4fd9-8391-ce3e1c73c4b5/1911e221-32e7-4aa1-805e-6cbecb9cf221"
-          (reference "J3") (unit 1)
+          (reference "J7") (unit 1)
         )
       )
@@
   (symbol (lib_id "Device:R") (at 119.38 110.998 0) (unit 1)
     (in_bom yes) (on_board yes) (dnp no) (fields_autoplaced)
-    (property "Reference" "RSens" (at 121.666 110.363 0)
+    (property "Reference" "RSens1" (at 121.666 110.363 0)
       (effects (font (size 1.27 1.27)) (justify left))
     )
@@
       (project "Grup3_Tarda_Projecte_Netejaparabrises"
         (path "/7ae78f34-680b-4fd9-8391-ce3e1c73c4b5/1911e221-32e7-4aa1-805e-6cbecb9cf221"
-          (reference "RSens") (unit 1)
+          (reference "RSens1") (unit 1)
         )
       )
@@
   (symbol (lib_id "Device:R_Potentiometer_Trim") (at 110.744 106.68 0) (unit 1)
     (in_bom yes) (on_board yes) (dnp no) (fields_autoplaced)
-    (property "Reference" "RPOT" (at 107.95 106.045 0)
+    (property "Reference" "RPOT1" (at 107.95 106.045 0)
       (effects (font (size 1.27 1.27)) (justify right))
     )
@@
       (project "Grup3_Tarda_Projecte_Netejaparabrises"
         (path "/7ae78f34-680b-4fd9-8391-ce3e1c73c4b5/1911e221-32e7-4aa1-805e-6cbecb9cf221"
-          (reference "RPOT") (unit 1)
+          (reference "RPOT1") (unit 1)
         )
       )
@@
   (symbol (lib_id "Device:C") (at 176.53 103.632 0) (unit 1)
     (in_bom yes) (on_board yes) (dnp no)
-    (property "Reference" "CDesOpam" (at 171.45 101.473 0)
+    (property "Reference" "CDesOpam1" (at 171.45 101.473 0)
       (effects (font (size 1.27 1.27)) (justify left))
     )
@@
       (effects (font (size 1.27 1.27)) (justify left))
     )
-    (property "Footprint" "" (at 177.4952 107.442 0)
+    (property "Footprint" "Capacitor_SMD:CP_Elec_4x3" (at 177.4952 107.442 0)
       (effects (font (size 1.27 1.27)) hide)
     )
@@
       (project "Grup3_Tarda_Projecte_Netejaparabrises"
         (path "/7ae78f34-680b-4fd9-8391-ce3e1c73c4b5/1911e221-32e7-4aa1-805e-6cbecb9cf221"
-          (reference "CDesOpam") (unit 1)
+          (reference "CDesOpam1") (unit 1)
         )
       )
@@
   (symbol (lib_id "Comparator:LM393") (at 141.478 103.886 0) (unit 1)
     (in_bom yes) (on_board yes) (dnp no) (fields_autoplaced)
-    (property "Reference" "U3" (at 141.478 94.742 0)
+    (property "Reference" "U2" (at 141.478 94.742 0)
       (effects (font (size 1.27 1.27)))
     )
@@
       (project "Grup3_Tarda_Projecte_Netejaparabrises"
         (path "/7ae78f34-680b-4fd9-8391-ce3e1c73c4b5/1911e221-32e7-4aa1-805e-6cbecb9cf221"
-          (reference "U3") (unit 1)
+          (reference "U2") (unit 1)
         )
       )
@@
   (symbol (lib_id "power:GND") (at 186.182 111.506 0) (unit 1)
     (in_bom yes) (on_board yes) (dnp no) (fields_autoplaced)
-    (property "Reference" "#PWR015" (at 186.182 117.856 0)
+    (property "Reference" "#PWR018" (at 186.182 117.856 0)
       (effects (font (size 1.27 1.27)) hide)
     )
@@
       (project "Grup3_Tarda_Projecte_Netejaparabrises"
         (path "/7ae78f34-680b-4fd9-8391-ce3e1c73c4b5/1911e221-32e7-4aa1-805e-6cbecb9cf221"
-          (reference "#PWR015") (unit 1)
+          (reference "#PWR018") (unit 1)
         )
       )
@@
   (symbol (lib_id "Comparator:LM393") (at 188.722 103.632 0) (unit 3)
     (in_bom yes) (on_board yes) (dnp no) (fields_autoplaced)
-    (property "Reference" "U3" (at 187.706 102.997 0)
+    (property "Reference" "U2" (at 187.706 102.997 0)
       (effects (font (size 1.27 1.27)) (justify left))
     )
@@
       (project "Grup3_Tarda_Projecte_Netejaparabrises"
         (path "/7ae78f34-680b-4fd9-8391-ce3e1c73c4b5/1911e221-32e7-4aa1-805e-6cbecb9cf221"
-          (reference "U3") (unit 3)
+          (reference "U2") (unit 3)
         )
       )
@@
   (symbol (lib_id "power:GND") (at 115.062 115.824 0) (unit 1)
     (in_bom yes) (on_board yes) (dnp no) (fields_autoplaced)
-    (property "Reference" "#PWR016" (at 115.062 122.174 0)
+    (property "Reference" "#PWR017" (at 115.062 122.174 0)
       (effects (font (size 1.27 1.27)) hide)
     )
@@
       (project "Grup3_Tarda_Projecte_Netejaparabrises"
         (path "/7ae78f34-680b-4fd9-8391-ce3e1c73c4b5/1911e221-32e7-4aa1-805e-6cbecb9cf221"
-          (reference "#PWR016") (unit 1)
-        )
-      )
+          (reference "#PWR017") (unit 1)
+        )
+      )
