File: Grup3_Tarda_Projecte_Netejaparabrises/Grup3_Tarda_Projecte_Netejaparabrises.kicad_pcb (KiCad board)
At the start: 4 copper layers, 162.4 x 126.5 mm, 89 parts, among them IC1 L78S05CV, IC2 PIC18F258-I_SO, J1 Screw_Terminal_01x02, J10 Screw_Terminal_01x02, J11 Screw_Terminal_01x02, J12 Screw_Terminal_01x02, J2 BOTONERA, J3 PROGRAMMING CON, J4 JP1, J5 DE9_Plug_MountingHoles, J6 DE9_Plug_MountingHoles, J7 CONEXIOSENSOR, J8 Screw_Terminal_01x02, J9 Screw_Terminal_01x02, K1 1393280-6, K2 1393280-6, K3 1393280-6, K4 1393280-6, K5 1393280-6, K6 1393280-6, K7 1393280-6, K8 1393280-6, K9 1393280-6, Q1 BC817-25_RF, Q2 BC817-25_RF, Q3 BC817-25_RF, Q4 BC817-25_RF, Q5 BC817-25_RF, Q6 BC817-25_RF, Q7 BC817-25_RF, U1 Value, U2 LM393, Y1 ABLS2-8.000MHZ-D4Y-T

Commit message: layout modificat a 2 capes
Parts:
- moved J7 5.04 mm to (96.8, 28.6), turned to 90 degrees
Routing:
- net +VCC: track 28.5 -> 276.9 mm, vias 9 -> 5
- net /Potencia/Vc_m1: track 99.0 -> 103.3 mm
- net EN2: track 66.2 -> 70.0 mm
- net EnableM2: track 18.8 -> 21.1 mm
- net DriverB1: track 74.1 -> 75.8 mm
- net GND: track 14.5 -> 13.9 mm
- added copper zone on B.Cu, net GND
- added copper zone on B.Cu, net GNDPWR
- added copper zone on F.Cu, net VBAT
- removed copper zone on In1.Cu, net +VCC
- removed copper zone on In2.Cu, net GND
- removed copper zone on In2.Cu, net GNDPWR
- removed copper zone on In1.Cu, net VBAT
Other:
- copper layers 4 -> 2
